Commit message: Fix optical frame orientation

File: aramis_description/robots/sensor_camera_usb_pioneer.urdf.xacro (robot description, xacro)
@@ -40,5 +40,5 @@
         <joint name="${name}_optical_joint" type="fixed">
             <!-- <origin xyz="-0.025 0.038 0.024" rpy="0 -1.57 0"/> -->
-            <origin xyz="0.025 0.026 0.024" rpy="0 0 0"/>
+            <origin xyz="0.025 0.026 0.024" rpy="0 0 3.14"/>
             <parent link="${name}_frame" />
             <child link="${name}_optical_frame" />
