Commit message: fix xacro

File: aramis_description/robots/pioneer3dx_body.xacro (robot description, xacro)
@@ -8,5 +8,5 @@
   <xacro:include filename="pioneer3dx_sonar.xacro"/>
   <xacro:include filename="pioneer3dx_plugins.xacro"/>
-  <xacro:macro xmlns:xacro="http://ros.org/wiki/xacro" name="pioneer3dx_body" params="name parent meshes">
+  <xacro:macro name="pioneer3dx_body" params="name parent meshes">
     <!-- base_link -->
     <link name="${parent}"/>
