Commit message: Add collision box with 0.01 m

File: aramis_description/robots/pioneer3dx_sonar.xacro (robot description, xacro)
@@ -27,5 +27,5 @@
       <origin xyz="0 0 0" rpy="0 0 0"/>
       <geometry>
-        <box size="0 0 0"/>
+        <box size="0.01 0.01 0.01"/>
       </geometry>
     </collision>

File: aramis_description/robots/pioneer3dx_swivel.xacro (robot description, xacro)
@@ -31,5 +31,5 @@
       <origin xyz="0 0 0" rpy="0 0 0"/>
       <geometry>
-        <box size="0 0 0"/>
+        <box size="0.01 0.01 0.01"/>
       </geometry>
     </collision>
@@ -98,5 +98,5 @@
       <origin xyz="0 0 0" rpy="0 0 0"/>
       <geometry>
-        <box size="0 0 0"/>
+        <box size="0.01 0.01 0.01"/>
       </geometry>
     </collision>

File: aramis_description/robots/pioneer3dx_wheel.xacro (robot description, xacro)
@@ -29,5 +29,5 @@
       <origin xyz="0 0 0" rpy="0 0 0"/>
       <geometry>
-        <box size="0 0 0"/>
+        <box size="0.01 0.01 0.01"/>
       </geometry>
     </collision>

Commit message: Fix color in gazzebo 7

File: aramis_description/robots/pioneer3dx_sonar.xacro (robot description, xacro)
@@ -18,5 +18,5 @@
       <origin xyz="0 0 0" rpy="0 0 0"/>
       <geometry name="pioneer_geom">
-        <mesh filename="${meshes}/back_sonar.stl"/>
+        <mesh filename="${meshes}/sonar.dae"/>
       </geometry>
       <material name="SonarYellow">

File: aramis_description/robots/pioneer3dx_swivel.xacro (robot description, xacro)
@@ -22,5 +22,5 @@
       <origin xyz="0 0 0" rpy="0 0 0"/>
       <geometry name="pioneer_geom">
-        <mesh filename="${meshes}/swivel.stl"/>
+        <mesh filename="${meshes}/swivel.dae"/>
       </geometry>
       <material name="swivel">
@@ -57,5 +57,5 @@
       <origin xyz="0 0 0" rpy="0 0 0"/>
       <geometry name="pioneer_geom">
-        <mesh filename="${meshes}/center_wheel.stl"/>
+        <mesh filename="${meshes}/center_wheel.dae"/>
       </geometry>
       <material name="WheelBlack">
@@ -89,5 +89,5 @@
       <origin xyz="0 0 0" rpy="0 0 0"/>
       <geometry name="pioneer_geom">
-        <mesh filename="${meshes}/center_hubcap.stl"/>
+        <mesh filename="${meshes}/center_hubcap.dae"/>
       </geometry>
       <material name="swivel">

File: aramis_description/robots/pioneer3dx_wheel.xacro (robot description, xacro)
@@ -20,5 +20,5 @@
       <origin xyz="0 0 0" rpy="0 0 0"/>
       <geometry name="pioneer_geom">
-        <mesh filename="${meshes}/${side}_hubcap.stl"/>
+        <mesh filename="${meshes}/${side}_hubcap.dae"/>
       </geometry>
       <material name="HubcapYellow">
@@ -52,5 +52,5 @@
       <origin xyz="0 0 0" rpy="0 0 0"/>
       <geometry name="pioneer_geom">
-        <mesh filename="${meshes}/${side}_wheel.stl"/>
+        <mesh filename="${meshes}/${side}_wheel.dae"/>
       </geometry>
       <material name="WheelBlack">
