Commit message: fix swivel wheel position

File: aramis_description/robots/pioneer3dx_swivel.xacro (robot description, xacro)
@@ -40,5 +40,5 @@
   <!-- Center Wheel -->
   <joint name="swivel_wheel_joint" type="continuous">
-    <origin xyz="-0.026 0 -0.016" rpy="0 0 0"/>
+    <origin xyz="-0.017 0 -0.016" rpy="0 0 0"/>
     <axis xyz="0 1 0"/>
     <anchor xyz="0 0 0"/>
