Commit message: Test in real robot

File: aramis_description/robots/aramis_description.xacro (robot description, xacro)
@@ -13,13 +13,19 @@
     <!--
     <joint name="pioneer2cyton" type="fixed">
-    	<origin xyz="0.08 0.071 0.004" rpy="0 0 0"/>
-    		<parent link="top"/>
-    		<child link="link0"/>
+        <origin xyz="0.08 0.071 0.004" rpy="0 0 0"/>
+            <parent link="top"/>
+            <child link="link0"/>
     </joint>
      -->
     <joint name="pioneer2suporte" type="fixed">
-    	<origin xyz="0.073 0.160 0.004" rpy="0 0 -1.57"/>
-    		<parent link="top"/>
-    		<child link="suporte_base"/>
+        <origin xyz="0.073 0.160 0.004" rpy="0 0 -1.57"/>
+           <parent link="top"/>
+           <child link="suporte_base"/>
+    </joint>
+    <link name="imu_link" />
+    <joint name="imu_joint" type="fixed" >
+        <origin xyz="0 0 0" rpy="0 0 0"/>
+        <parent link="top" />
+        <child link="imu_link" />
     </joint>
     <kinect_camera_v0 name="kinect" parent="suporte_kinect">

Commit message: remove suporte and new kinect location

File: aramis_description/robots/aramis_description.xacro (robot description, xacro)
@@ -2,7 +2,7 @@
 <robot xmlns:xacro="http://ros.org/wiki/xacro" name="aramis_description">
     <xacro:include filename="$(find aramis_description)/robots/pioneer3dx.xacro"/>
-    <xacro:include filename="$(find aramis_description)/robots/suporte_aramis_description.URDF"/>
+    <!-- <xacro:include filename="$(find aramis_description)/robots/suporte_aramis_description.URDF"/> -->
     <xacro:include filename="$(find aramis_description)/robots/sensor_sonar_pioneer.urdf.xacro"/>
-    <xacro:include filename="$(find aramis_description)/robots/sensor_camera_usb_pioneer.urdf.xacro"/>
+    <!-- <xacro:include filename="$(find aramis_description)/robots/sensor_camera_usb_pioneer.urdf.xacro"/> -->
     <xacro:include filename="$(find pr2_description)/urdf/sensors/kinect_camera.urdf.xacro" />
     <xacro:include filename="$(find pr2_description)/urdf/common.xacro" />
@@ -18,14 +18,14 @@
     </joint>
      -->
-    <joint name="pioneer2suporte" type="fixed">
+<!--     <joint name="pioneer2suporte" type="fixed">
         <origin xyz="0.073 0.160 0.004" rpy="0 0 -1.57"/>
             <parent link="top"/>
             <child link="suporte_base"/>
-    </joint>
-    <kinect_camera_v0 name="kinect" parent="suporte_kinect">
+    </joint> -->
+    <kinect_camera_v0 name="kinect" parent="top">
         <!-- <origin rpy="0 -3.9246 1.57"  xyz="0.170 0.067 -0.035"/> -->
-        <origin rpy="0 1.57 1.57"  xyz="0.170 0.087 0.0"/>
+        <origin rpy="0 0 0"  xyz="0.200 0.0 0.05"/>
     </kinect_camera_v0>
-    <camera_usb name="usb_camera" parent="suporte_kinect">
+    <camera_usb name="usb_camera" parent="top">
         <!-- //<origin rpy="0 -3.9246 1.57"  xyz="0.170 0.067 -0.035"/> -->
         <origin rpy="1.57 0 3.14"  xyz="0.275 0.0 0.060"/>

Commit message: update

File: aramis_description/robots/aramis_description.xacro (robot description, xacro)
@@ -2,8 +2,8 @@
 <robot xmlns:xacro="http://ros.org/wiki/xacro" name="aramis_description">
     <xacro:include filename="$(find aramis_description)/robots/pioneer3dx.xacro"/>
-    <!-- <xacro:include filename="$(find aramis_description)/robots/suporte_aramis_description.URDF"/> -->
+    <xacro:include filename="$(find aramis_description)/robots/suporte_aramis_description.urdf"/>
     <xacro:include filename="$(find aramis_description)/robots/sensor_sonar_pioneer.urdf.xacro"/>
     <!-- <xacro:include filename="$(find aramis_description)/robots/sensor_camera_usb_pioneer.urdf.xacro"/> -->
-    <xacro:include filename="$(find pr2_description)/urdf/sensors/kinect_camera.urdf.xacro" />
+    <!-- <xacro:include filename="$(find pr2_description)/urdf/sensors/kinect_camera.urdf.xacro" /> -->
     <xacro:include filename="$(find pr2_description)/urdf/common.xacro" />
     <!-- <xacro:p3dx_front suffix="left" reflect="1"/> -->
@@ -18,12 +18,12 @@
     </joint>
      -->
-<!--     <joint name="pioneer2suporte" type="fixed">
+    <joint name="pioneer2suporte" type="fixed">
         <origin xyz="0.073 0.160 0.004" rpy="0 0 -1.57"/>
             <parent link="top"/>
             <child link="suporte_base"/>
-    </joint> -->
-    <kinect_camera_v0 name="kinect" parent="top">
-        <!-- <origin rpy="0 -3.9246 1.57"  xyz="0.170 0.067 -0.035"/> -->
-        <origin rpy="0 0 0"  xyz="0.200 0.0 0.05"/>
+    </joint>
+    <kinect_camera_v0 name="kinect" parent="suporte_kinect">
+        <origin rpy="0 -3.9246 1.57"  xyz="0.170 0.067 -0.035"/>
+        <!-- <origin rpy="0 0 0"  xyz="0.200 0.0 0.05"/> -->
     </kinect_camera_v0>
     <camera_usb name="usb_camera" parent="top">
@@ -31,4 +31,5 @@
         <origin rpy="1.57 0 3.14"  xyz="0.275 0.0 0.060"/>
     </camera_usb>
+<!--
     <sonar_pioneer name="sonar_0" parent="base_link">
         <origin xyz="0.069 0.130 0.209" rpy="0 0 1.5708"/>
@@ -54,5 +55,5 @@
     <sonar_pioneer name="sonar_7" parent="base_link">
         <origin xyz="0.069 -0.130 0.209" rpy="0 0 -1.5708"/>
-    </sonar_pioneer>
+    </sonar_pioneer> -->
     <link name="back_sonar_range_frame" />
     <joint name="back_sonar_range_joint" type="fixed">

File: aramis_description/robots/pioneer3dx_chassis.xacro (robot description, xacro)
@@ -11,7 +11,7 @@
   <link name="${name}">
     <visual name="chassis_visual">
-      <origin xyz="-0.045 0 0.148" rpy="0 0 0"/>
+      <origin xyz="-0.0 0 0.0" rpy="0 0 0"/>
       <geometry name="pioneer_geom">
-        <mesh filename="${meshes}/chassis.stl"/>
+        <mesh filename="${meshes}/chassis_mesh.dae"/>
       </geometry>
       <material name="ChassisRed">
@@ -20,7 +20,7 @@
     </visual>
     <collision>
-      <origin xyz="-0.045 0 0.148" rpy="0 0 0"/>
+      <origin xyz="-0.0 0 0.148" rpy="0 0 0"/>
       <geometry>
-        <mesh filename="${meshes}/chassis.stl"/>
+        <mesh filename="${meshes}/chassis_mesh.dae"/>
       </geometry>
     </collision>
@@ -32,5 +32,5 @@
   <!-- Top -->
   <joint name="${name}_top_joint" type="fixed">
-    <origin xyz="-0.045 0 0.234" rpy="0 0 0"/>
+    <origin xyz="-0.045 0 0.238" rpy="0 0 0"/>
     <parent link="${name}"/>
     <child link="top"/>
@@ -38,7 +38,7 @@
   <link name="top">
     <visual>
-      <origin xyz="0 0 0" rpy="0 0 0"/>
+      <origin xyz="0 0 0.0" rpy="0 0 0"/>
       <geometry name="top_geom">
-        <mesh filename="${meshes}/top.stl"/>
+        <mesh filename="${meshes}/top_mesh2.dae"/>
       </geometry>
       <material name="TopBlack">
@@ -49,5 +49,5 @@
     <origin xyz="0.0 0 0.0" rpy="0 0 0"/>
       <geometry>
-        <mesh filename="${meshes}/top.stl"/>
+        <mesh filename="${meshes}/top_mesh2.dae"/>
       </geometry>
     </collision>

File: aramis_description/robots/pioneer3dx_plugins.xacro (robot description, xacro)
@@ -6,5 +6,5 @@
           <robotNamespace></robotNamespace>
           <jointName>chassis_swivel_joint, swivel_wheel_joint, left_hub_joint, right_hub_joint</jointName>
-          <updateRate>10.0</updateRate>
+          <updateRate>25.0</updateRate>
           <alwaysOn>true</alwaysOn>
         </plugin>
@@ -15,10 +15,10 @@
         <plugin name="differential_drive_controller" filename="libgazebo_ros_diff_drive.so">
             <rosDebugLevel>Debug</rosDebugLevel>
-            <robotNamespace>/</robotNamespace>
+            <!-- <robotNamespace>/</robotNamespace> -->
             <publishWheelTF>false</publishWheelTF>
             <publishWheelJointState>true</publishWheelJointState>
             <alwaysOn>true</alwaysOn>
-            <leftJoint>left_hub_joint</leftJoint>
-            <rightJoint>right_hub_joint</rightJoint>
+            <leftJoint>right_hub_joint</leftJoint>
+            <rightJoint>left_hub_joint</rightJoint>
             <wheelSeparation>0.3</wheelSeparation>
             <wheelDiameter>0.18</wheelDiameter>
@@ -31,4 +31,7 @@
             <odometrySource>world</odometrySource>
             <robotBaseFrame>base_link</robotBaseFrame>
+            <covariance_x>1</covariance_x>
+            <covariance_y>1</covariance_y>
+            <covariance_yaw>1</covariance_yaw>
             <updateRate>50.0</updateRate>
             <publishTf>1</publishTf>

File: aramis_description/robots/suporte_aramis_description.urdf (robot description, URDF)
Before this commit: robot suporte_aramis_description, 7 links, 6 joints
Links:
- link suporte_armControl: geometry collision mesh filename=package://aramis_description/meshes/suporte_armControl_mesh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; visual mesh filename=package://aramis_description/meshes/suporte_armControl_mesh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
- link suporte_base: geometry collision mesh filename=package://aramis_description/meshes/suporte_base_mesh.dae; visual mesh filename=package://aramis_description/meshes/suporte_base_mesh.dae
- link suporte_kinect: geometry collision mesh filename=package://aramis_description/meshes/suporte_kinect_mesh2.dae; visual mesh filename=package://aramis_description/meshes/suporte_kinect_mesh2.dae
- link tampa1: geometry collision mesh filename=package://aramis_description/meshes/tampa1_mesh.dae; visual mesh filename=package://aramis_description/meshes/tampa1_mesh.dae
- link tampa2: geometry collision mesh filename=package://aramis_description/meshes/tampa2_mesh.dae; visual mesh filename=package://aramis_description/meshes/tampa2_mesh.dae
- link tampa3: geometry collision mesh filename=package://aramis_description/meshes/tampa3_mesh.dae; visual mesh filename=package://aramis_description/meshes/tampa3_mesh.dae
- link tampa4: geometry collision mesh filename=package://aramis_description/meshes/tampa4_mesh.dae; visual mesh filename=package://aramis_description/meshes/tampa4_mesh.dae
Joints:
- joint armControl: origin xyz=0.03 -0.043 0.145 rpy=1.5708 0 0 -> xyz=0.161 -0.0743 0.1569 rpy=1.5708 0 0
- joint kinect_joint: origin xyz=0 -0.0429999999999997 0.6 rpy=1.5707963267949 0 0 -> xyz=0.161 -0.074 0.615 rpy=1.5707963267949 0 0
